File: Ultramarine_fuse/Ultramarine_fuse.kicad_pcb (KiCad board)
At the start: 2 copper layers, 123 parts, among them J1 Conn_01x04_Female, J2 Conn_01x04_Female, SW1 SW_Push, SW10 SW_Push, SW11 SW_Push, SW12 SW_Push, SW13 SW_Push, SW14 SW_Push, SW15 SW_Push, SW16 SW_Push, SW17 SW_Push, SW18 SW_Push, SW19 SW_Push, SW2 SW_Push, SW20 SW_Push, SW21 SW_Push, SW22 SW_Push, SW23 SW_Push, SW24 SW_Push, SW25 SW_Push, SW26 SW_Push, SW27 SW_Push, SW28 SW_Push, SW29 SW_Push, SW3 SW_Push, SW30 SW_Push, SW31 SW_Push, SW32 SW_Push, SW33 SW_Push, SW34 SW_Push, SW35 SW_Push, SW36 SW_Push, SW4 SW_Push, SW5 SW_Push, SW6 SW_Push, SW7 SW_Push, SW8 SW_Push, SW9 SW_Push, U1 Pro_Micro, U10 SK6812mini, U11 SK6812mini, U12 SK6812mini, U13 SK6812mini, U14 SK6812mini, U15 SK6812mini, U16 SK6812mini, U17 SK6812mini, U18 SK6812mini, U19 SK6812mini, U2 SK6812mini, U20 SK6812mini, U21 SK6812mini, U22 SK6812mini, U23 SK6812mini, U24 SK6812mini, U25 SK6812mini, U26 SK6812mini, U27 SK6812mini, U28 SK6812mini, U29 SK6812mini, U3 SK6812mini, U30 SK6812mini, U31 SK6812mini, U32 SK6812mini, U33 SK6812mini, U34 SK6812mini, U35 SK6812mini, U36 SK6812mini, U4 SK6812mini, U5 SK6812mini, U6 SK6812mini, U7 SK6812mini, U8 SK6812mini, U9 SK6812mini

Commit message: nothing special
Parts:
- removed G***: LOGO, Ultramarine_fuse:logo
- moved R1 214.4 mm to (104.0, 211.5)
- moved J2 199.1 mm to (266.1, 39.4), turned to 270 degrees
- moved U16 197.7 mm to (310.0, 150.0), turned to 180 degrees
- moved U17 196.2 mm to (300.0, 150.0), turned to 180 degrees
- moved J1 192.9 mm to (264.2, 31.1), turned to 90 degrees
- moved U15 189.8 mm to (310.0, 140.0)
- moved SW36 183.9 mm to (267.3, 47.0), turned to 180 degrees
- moved U14 165.0 mm to (300.0, 140.0)
- moved D8 153.1 mm to (134.5, 22.5), turned to 180 degrees
- moved U13 147.6 mm to (290.0, 140.0)
- moved D22 143.8 mm to (134.5, 60.5), turned to 180 degrees
- moved U6 142.4 mm to (270.0, 130.0), turned to 180 degrees
- moved D14 141.8 mm to (248.5, 25.0), turned to 180 degrees
- moved D35 137.3 mm to (259.8, 91.8), turned to 240 degrees
- moved U4 134.2 mm to (210.5, 4.00), turned to 180 degrees
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Connections:
- SW1 pad 1: Net-(SW1-Pad1) -> /Col0
- SW10 pad 1: Net-(SW10-Pad1) -> /Col2
- SW11 pad 1: Net-(SW11-Pad1) -> /Col3
- SW12 pad 1: Net-(SW12-Pad1) -> /Col4
- SW13 pad 1: Net-(SW13-Pad1) -> /Col5
- SW14 pad 1: Net-(SW14-Pad1) -> /Col6
- SW15 pad 1: Net-(SW15-Pad1) -> /Col0
- SW16 pad 1: Net-(SW16-Pad1) -> /Col1
- SW17 pad 1: Net-(SW17-Pad1) -> /Col2
- SW18 pad 1: Net-(SW18-Pad1) -> /Col3
- SW19 pad 1: Net-(SW19-Pad1) -> /Col4
- SW2 pad 1: Net-(SW2-Pad1) -> /Col1
- SW20 pad 1: Net-(SW20-Pad1) -> /Col5
- SW21 pad 1: Net-(SW21-Pad1) -> /Col6
- SW22 pad 1: Net-(SW22-Pad1) -> /Col0
- SW23 pad 1: Net-(SW23-Pad1) -> /Col1
- SW24 pad 1: Net-(SW24-Pad1) -> /Col2
- SW25 pad 1: Net-(SW25-Pad1) -> /Col3
- SW26 pad 1: Net-(SW26-Pad1) -> /Col4
- SW27 pad 1: Net-(SW27-Pad1) -> /Col5
- SW28 pad 1: Net-(SW28-Pad1) -> /Col6
- SW3 pad 1: Net-(SW3-Pad1) -> /Col2
- SW4 pad 1: Net-(SW4-Pad1) -> /Col3
- SW5 pad 1: Net-(SW5-Pad1) -> /Col4
- SW6 pad 1: Net-(SW6-Pad1) -> /Col5
- SW7 pad 1: Net-(SW7-Pad1) -> /Col6
- SW8 pad 1: Net-(SW8-Pad1) -> /Col0
- SW9 pad 1: Net-(SW9-Pad1) -> /Col1
- U10 pad 2: Net-(U10-Pad2) -> GND
- U10 pad 4: Net-(U10-Pad4) -> VCC
- U11 pad 2: Net-(U11-Pad2) -> GND
- U11 pad 4: Net-(U11-Pad4) -> VCC
- U12 pad 2: Net-(U12-Pad2) -> GND
- U12 pad 4: Net-(U12-Pad4) -> VCC
- U13 pad 2: Net-(U13-Pad2) -> GND
- U13 pad 4: Net-(U13-Pad4) -> VCC
- U14 pad 2: Net-(U14-Pad2) -> GND
- U14 pad 4: Net-(U14-Pad4) -> VCC
- U15 pad 2: Net-(U15-Pad2) -> GND
- U15 pad 4: Net-(U15-Pad4) -> VCC
- U23 pad 2: Net-(U23-Pad2) -> GND
- U23 pad 4: Net-(U23-Pad4) -> VCC
- U24 pad 2: Net-(U24-Pad2) -> GND
- U24 pad 4: Net-(U24-Pad4) -> VCC
- U25 pad 2: Net-(U25-Pad2) -> GND
- U25 pad 4: Net-(U25-Pad4) -> VCC
- U26 pad 2: Net-(U26-Pad2) -> GND
- U26 pad 4: Net-(U26-Pad4) -> VCC
- U27 pad 2: Net-(U27-Pad2) -> GND
- U27 pad 4: Net-(U27-Pad4) -> VCC
- U28 pad 2: Net-(U28-Pad2) -> GND
- U28 pad 4: Net-(U28-Pad4) -> VCC
- U29 pad 2: Net-(U29-Pad2) -> GND
- U29 pad 4: Net-(U29-Pad4) -> VCC
- U3 pad 4: Net-(U3-Pad4) -> VCC
- U31 pad 2: Net-(U31-Pad2) -> GND
- U32 pad 2: Net-(U32-Pad2) -> GND
- U33 pad 2: Net-(U33-Pad2) -> GND
- U34 pad 2: Net-(U34-Pad2) -> GND
- U35 pad 2: Net-(U35-Pad2) -> GND
- U36 pad 2: Net-(U36-Pad2) -> GND
- U4 pad 4: Net-(U4-Pad4) -> VCC
- U5 pad 4: Net-(U5-Pad4) -> VCC
- U6 pad 4: Net-(U6-Pad4) -> VCC
- U7 pad 4: Net-(U7-Pad4) -> VCC
Routing:
- net /Col0: track 14.5 -> 297.9 mm, vias 0 -> 2
- net /Col1: track 14.5 -> 280.7 mm, vias 0 -> 2
- net /Row4: track 17.0 -> 278.5 mm, vias 0 -> 7
- net /Col2: track 14.5 -> 261.6 mm, vias 0 -> 2
- net /Col3: track 14.5 -> 249.6 mm, vias 0 -> 2
- net /Col4: track 14.5 -> 237.3 mm, vias 0 -> 2
- net /Col5: track 14.5 -> 221.4 mm, vias 0 -> 2
- net /Col6: track 14.5 -> 207.8 mm, vias 0 -> 2
- net /Row1: track 17.0 -> 184.9 mm, vias 0 -> 7
- net /Row2: track 17.0 -> 184.9 mm, vias 0 -> 1
- net /Row0: track 17.0 -> 179.2 mm, vias 0 -> 6
- net /Row3: track 17.0 -> 101.2 mm, vias 0 -> 1
- net GND: track 0.00 -> 52.9 mm
- net Net-(D32-Pad2): track 0.00 -> 25.1 mm
- net Net-(D9-Pad2): track 0.00 -> 25.1 mm
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
Commit message: PCB making without Charging unit is completed
Parts:
- added G***: LOGO, Ultramarine_fuse:logo, F.Cu at (111.8, 94.6)
- J1: footprint Connector_PinSocket_2.54mm:PinSocket_1x04_P2.54mm_Vertical -> Basic_THT:4pin_A
- JP5, JP6, JP7, JP8: moved to B.Cu
- moved U16 272.5 mm to (43.0, 95.5), turned to 0 degrees
- moved U30 269.5 mm to (43.0, 133.5), turned to 0 degrees
- moved U17 244.2 mm to (62.0, 95.5), turned to 0 degrees
- moved U31 240.8 mm to (62.0, 133.5), turned to 0 degrees
- moved U18 217.2 mm to (81.0, 91.0), turned to 0 degrees
- moved U9 216.5 mm to (43.0, 76.5), turned to 180 degrees
- moved U32 213.0 mm to (81.0, 129.0), turned to 0 degrees
- moved U23 211.9 mm to (43.0, 114.5), turned to 180 degrees
- moved U2 210.7 mm to (43.0, 57.5), turned to 0 degrees
- moved U10 207.9 mm to (62.0, 76.5), turned to 180 degrees
- moved U24 203.2 mm to (62.0, 114.5), turned to 180 degrees
- moved U11 200.9 mm to (81.0, 72.0), turned to 180 degrees
- moved U25 195.5 mm to (81.0, 110.0), turned to 180 degrees
- moved U12 193.5 mm to (100.0, 69.0), turned to 180 degrees
- moved U19 190.4 mm to (100.0, 88.0), turned to 0 degrees
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Routing:
- net VCC: track 29.0 -> 1498.6 mm, vias 2 -> 37
- net /Row3: track 101.2 -> 250.2 mm, vias 1 -> 7
- net /~RESET: track 14.5 -> 83.8 mm
- net Net-(U16-Pad1): track 0.00 -> 68.8 mm, vias 0 -> 2
- net Net-(U2-Pad1): track 0.10 -> 68.1 mm, vias 0 -> 2
- net /data: track 17.0 -> 71.7 mm, vias 2 -> 3
- net /SCL: track 17.0 -> 63.6 mm, vias 0 -> 2
- net Net-(U32-Pad3): track 0.00 -> 44.6 mm, vias 0 -> 1
- net /SDA: track 17.0 -> 60.8 mm, vias 0 -> 2
- net Net-(U29-Pad1): track 0.00 -> 42.8 mm, vias 0 -> 2
- net Net-(U35-Pad3): track 0.00 -> 40.6 mm, vias 0 -> 2
- net Net-(U15-Pad1): track 0.00 -> 38.3 mm, vias 0 -> 2
- net Net-(U33-Pad3): track 0.00 -> 35.9 mm, vias 0 -> 1
- net Net-(U31-Pad3): track 0.00 -> 32.9 mm, vias 0 -> 1
- net /Row4: track 278.5 -> 309.2 mm
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- added copper zone on B.Cu, net GND
- added copper zone on F.Cu, net GND
Other:
- board outline added: 152.5 x 126 mm
- board text added: "Designed by Chrodream ~ Board Rev. 1.0"
- board text added: "Ultramarine Igniter"

Commit message: made for test printing
Parts:
- added C1: 4.7u, Basic_SOP:C1608, F.Cu at (173.4, 104.8)
- added C2: 4.7u, Basic_SOP:C1608, F.Cu at (179.7, 109.0)
- added C3: 0.1u, Basic_SOP:C1608, F.Cu at (179.7, 107.0)
- added C4: 4.7u, Basic_SOP:C1608, F.Cu at (168.6, 114.0)
- added D37: LED, Basic_SOP:LED1608, F.Cu at (178.8, 111.5)
- added J3: Conn_01x02_Male, Basic_THT:S2B-PH-K-S, F.Cu at (174.9, 113.6)
- added J4: Conn_01x02_Male, Basic_THT:S2B-PH-K-S, F.Cu at (164.6, 113.8)
- added Q1: AO3401A, Package_TO_SOT_SMD:SOT-23, F.Cu at (175.6, 108.3)
- added Q2: AO3400A, Package_TO_SOT_SMD:SOT-23, F.Cu at (170.6, 110.7)
- added Q3: AO3400A, Package_TO_SOT_SMD:SOT-23, F.Cu at (178.7, 103.8)
- added R1: 2.2K, Basic_SOP:1608, F.Cu at (160.0, 110.4)
- added R2: 330, Basic_SOP:1608, F.Cu at (165.9, 107.3)
- added R4: 100, Basic_SOP:1608, F.Cu at (160.0, 112.7)
- added R5: 100K, Basic_SOP:1608, F.Cu at (174.0, 102.6)
- added R6: 0.1, Basic_SOP:1608, F.Cu at (165.9, 109.6)
- added R7: 1K, Basic_SOP:1608, F.Cu at (170.9, 107.3)
- added SW37: SW_DPDT_x2, Basic_THT:SlideSW-3, F.Cu at (161.6, 103.0)
- added U37: MCP73831, Package_TO_SOT_SMD:SOT-23-5_HandSoldering, F.Cu at (168.6, 103.8)
- added U38: DW01A-G, Package_TO_SOT_SMD:SOT-23-6_Handsoldering, F.Cu at (160.5, 106.9)
- R10: renamed from R4; value R -> 10K
- R8: renamed from R2; value R -> 330
- R9: renamed from R3; value R -> 10K
Routing:
- net VCC: track 1498.6 -> 1503.4 mm

Commit message: fix circuit
Parts:
- removed D1, D15, D22, D28, D29, D30, D31, D32, D33, D34, D35, D8: D, Basic_SOP:1N4148
- removed SW1, SW15, SW22, SW28, SW29, SW30, SW31, SW32, SW33, SW34, SW35, SW8: SW_Push, Switch_Keyboard_Cherry_MX:MX-Kailh
- removed U16, U2, U23, U29, U30, U31, U32, U33, U34, U35, U36, U9: SK6812mini, Basic_SOP:SK6812mini
- J4: moved to B.Cu
- moved SW37 22.5 mm to (183.5, 108.0), turned to 90 degrees
- moved R1 17.6 mm to (175.9, 102.9), turned to 90 degrees
- moved Q3 17.4 mm to (161.3, 104.1), turned to 180 degrees
- moved C4 16.3 mm to (181.6, 104.1), turned to 90 degrees
- moved C3 14.6 mm to (165.7, 111.1)
- moved C2 14.2 mm to (166.4, 113.7)
- moved U37 10.6 mm to (178.8, 101.0), turned to 90 degrees
- moved Q2 9.71 mm to (161.3, 108.0), turned to 270 degrees
- moved R6 8.82 mm to (158.1, 105.4), turned to 270 degrees
- moved J4 6.97 mm to (171.4, 112.4)
- moved R2 6.17 mm to (170.2, 102.9), turned to 270 degrees
- moved R7 5.13 mm to (168.3, 102.9), turned to 270 degrees
- moved J3 4.69 mm to (171.4, 110.5), turned to 180 degrees
- moved U38 4.65 mm to (165.1, 106.9), turned to 270 degrees
- moved Q1 4.29 mm to (179.7, 107.0), turned to 90 degrees
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Routing:
- net VCC: track 1503.4 -> 996.6 mm, vias 37 -> 28
- net /Row4: track 309.2 -> 72.2 mm, vias 7 -> 0
- net /Col0: track 297.4 -> 146.0 mm
- net /Bat+: track 0.00 -> 82.2 mm
- net Net-(C2-Pad1): track 0.00 -> 52.9 mm
- net Net-(U2-Pad1): track 68.1 -> 16.7 mm, vias 2 -> 0
- net Net-(U16-Pad1): track 68.8 -> 18.0 mm, vias 2 -> 0
- net /Row3: track 250.2 -> 199.6 mm, vias 7 -> 6
- net /Col6: track 205.1 -> 160.1 mm
- net Net-(U32-Pad3): track 44.6 -> 0.00 mm, vias 1 -> 0
- net Net-(U29-Pad1): track 42.8 -> 0.00 mm, vias 2 -> 0
- net Net-(U35-Pad3): track 40.6 -> 0.00 mm, vias 2 -> 0
- net Net-(U33-Pad3): track 35.9 -> 0.00 mm, vias 1 -> 0
- net /Col1: track 280.9 -> 314.2 mm
- net Net-(U31-Pad3): track 32.9 -> 0.00 mm, vias 1 -> 0
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Other:
- board size 152.5 x 126 mm -> 134.5 x 94.2 mm
- board text removed: "Designed by Chrodream ~ Board Rev. 1.0"
- board text removed: "Ultramarine Igniter"
