File: Ultramarine_fuse/Ultramarine_fuse.kicad_pcb (KiCad board)
At the start: 2 copper layers, 152.5 x 126 mm, 132 parts, among them J1 Conn_01x04_Female, J2 Conn_01x04_Female, J3 Conn_01x02_Female, SW1 SW_Push, SW10 SW_Push, SW11 SW_Push, SW12 SW_Push, SW13 SW_Push, SW14 SW_Push, SW15 SW_Push, SW16 SW_Push, SW17 SW_Push, SW18 SW_Push, SW19 SW_Push, SW2 SW_Push, SW20 SW_Push, SW21 SW_Push, SW22 SW_Push, SW23 SW_Push, SW24 SW_Push, SW25 SW_Push, SW26 SW_Push, SW27 SW_Push, SW28 SW_Push, SW29 SW_Push, SW3 SW_Push, SW30 SW_Push, SW31 SW_Push, SW32 SW_Push, SW33 SW_Push, SW34 SW_Push, SW35 SW_Push, SW36 SW_Push, SW4 SW_Push, SW5 SW_Push, SW6 SW_Push, SW7 SW_Push, SW8 SW_Push, SW9 SW_Push, U1 BLE-Micro-Pro, U10 SK6812mini, U11 SK6812mini, U12 SK6812mini, U13 SK6812mini, U14 SK6812mini, U15 SK6812mini, U16 SK6812mini, U17 SK6812mini, U18 SK6812mini, U19 SK6812mini, U2 SK6812mini, U20 SK6812mini, U21 SK6812mini, U22 SK6812mini, U23 SK6812mini, U24 SK6812mini, U25 SK6812mini, U26 SK6812mini, U27 SK6812mini, U28 SK6812mini, U29 SK6812mini, U3 SK6812mini, U30 SK6812mini, U31 SK6812mini, U32 SK6812mini, U33 SK6812mini, U34 SK6812mini, U35 SK6812mini, U36 SK6812mini, U37 TP4056, U4 SK6812mini, U5 SK6812mini, U6 SK6812mini, U7 SK6812mini, U8 SK6812mini, U9 SK6812mini

Commit message: add 3v3 regulator
Parts:
- added G***: LOGO, Ultramarine_fuse:powered_by_qmk, B.Cu at (94.0, 133.0)
- added REF**: Stabilizer_Cherry_MX_2u, Mounting_Keyboard_Stabilizer:Stabilizer_Cherry_MX_2u, F.Cu at (168.2, 140.8)
- added U38: NJM2845, Package_TO_SOT_SMD:TO-252-2, B.Cu at (163.0, 109.0)
- added U39: NJM2845, Package_TO_SOT_SMD:TO-252-2, F.Cu at (163.0, 109.0)
- moved R8 32.1 mm to (195.3, 106.0)
- moved D36 29.3 mm to (193.0, 106.0)
- moved R10 25.5 mm to (169.2, 84.8), turned to 0 degrees
- moved R9 22.1 mm to (169.2, 87.1), turned to 0 degrees
- moved SW36 4.06 mm to (153.5, 46.0)
Connections:
- JP14 pad 2: /Bat+ -> Net-(JP14-Pad2)
- JP16 pad 2: /Bat+ -> Net-(JP14-Pad2)
Routing:
- net GND: track 162.6 -> 0.00 mm, vias 1 -> 0
- net VCC: track 112.0 -> 0.00 mm, vias 1 -> 0
- net /Bat+: track 105.4 -> 0.00 mm, vias 1 -> 0
- net /SDA: track 40.1 -> 0.00 mm, vias 2 -> 0
- net /SCL: track 33.9 -> 0.00 mm, vias 2 -> 0
- net Net-(J1-Pad4): track 5.64 -> 0.00 mm
- net Net-(J1-Pad1): track 5.64 -> 0.00 mm
- net Net-(JP13-Pad1): track 4.90 -> 0.00 mm
- net Net-(JP11-Pad2): track 4.90 -> 0.00 mm
- net Net-(JP15-Pad1): track 4.90 -> 0.00 mm
- net Net-(JP10-Pad2): track 4.90 -> 0.00 mm
- net Net-(J1-Pad3): track 4.59 -> 0.00 mm
- net Net-(J1-Pad2): track 4.59 -> 0.00 mm
- net Net-(J3-Pad1): track 4.19 -> 0.00 mm
- net Net-(J3-Pad2): track 3.68 -> 0.00 mm
Other:
- outline, holes or cut-outs redrawn
- board text added: "Ultramarine igniter Rev 1.0 Made by Chrodream"
