File: Ultramarine_fuse/Ultramarine_fuse.sch (KiCad schematic (older format))
At the start: 138 parts, among them J1 Conn_01x04_Female, J2 Conn_01x04_Female, J3 Conn_01x02_Male, Q1 AO3401A, SW1 SW_Push, SW10 SW_Push, SW11 SW_Push, SW12 SW_Push, SW13 SW_Push, SW14 SW_Push, SW15 SW_Push, SW16 SW_Push, SW17 SW_Push, SW18 SW_Push, SW19 SW_Push, SW2 SW_Push, SW20 SW_Push, SW21 SW_Push, SW22 SW_Push, SW23 SW_Push, SW24 SW_Push, SW25 SW_Push, SW26 SW_Push, SW27 SW_Push, SW28 SW_Push, SW29 SW_Push, SW3 SW_Push, SW30 SW_Push, SW31 SW_Push, SW32 SW_Push, SW33 SW_Push, SW34 SW_Push, SW35 SW_Push, SW36 SW_Push, SW4 SW_Push, SW5 SW_Push, SW6 SW_Push, SW7 SW_Push, SW8 SW_Push, SW9 SW_Push, U1 Pro_Micro, U10 SK6812mini, U11 SK6812mini, U12 SK6812mini, U13 SK6812mini, U14 SK6812mini, U15 SK6812mini, U16 SK6812mini, U17 SK6812mini, U18 SK6812mini, U19 SK6812mini, U2 SK6812mini, U20 SK6812mini, U21 SK6812mini, U22 SK6812mini, U23 SK6812mini, U24 SK6812mini, U25 SK6812mini, U26 SK6812mini, U27 SK6812mini, U28 SK6812mini, U29 SK6812mini, U3 SK6812mini, U30 SK6812mini, U31 SK6812mini, U32 SK6812mini, U33 SK6812mini, U34 SK6812mini, U35 SK6812mini, U36 SK6812mini, U37 MCP73831, U38 DW01A-G, U39 FS8205A, U4 SK6812mini, U5 SK6812mini, U6 SK6812mini, U7 SK6812mini, U8 SK6812mini, U9 SK6812mini

Commit message: fixed charge circuit for TP4056
Parts:
- removed C1, C2, C4: 4.7u, Basic_SOP:C1608, symbol Device:C
- removed C3: 0.1u, Basic_SOP:C1608, symbol Device:C
- removed D37: LED, symbol Device:LED
- removed D37: D_Schottky, symbol Device:D_Schottky
- removed J3: Conn_01x02_Male, symbol Connector:Conn_01x02_Male
- removed Q1: AO3401A, Package_TO_SOT_SMD:SOT-23, symbol Transistor_FET:AO3401A
- removed R1: 2.2K, Basic_SOP:1608, symbol Device:R
- removed R2: 330, Basic_SOP:1608, symbol Device:R
- removed R4: 100, Basic_SOP:1608, symbol Device:R
- removed R5: 100K, Basic_SOP:1608, symbol Device:R
- removed R6: 0.1, Basic_SOP:1608, symbol Device:R
- removed R7: 1K, Basic_SOP:1608, symbol Device:R
- removed U1: Pro_Micro, ATMega:Pro-Micro, symbol ATMega:Pro_Micro
- removed U37: MCP73831, symbol Basic_SOP:MCP73831
- removed U38: DW01A-G, symbol Basic_SOP:DW01A-G
- removed U39: FS8205A, symbol Basic_SOP:FS8205A
- added J3: Conn_01x02_Female, Basic_THT:S2B-PH-K-S, symbol Connector:Conn_01x02_Female
- added JP10, JP11, JP12, JP13, JP14, JP15, JP16, JP9: Jumper, Jumper:SolderJumper-2_P1.3mm_Open_RoundedPad1.0x1.5mm, symbol Device:Jumper
- added U1: BLE-Micro-Pro, ATMega:BLE-Micro-Pro, symbol ATMega:BLE-Micro-Pro
- added U37: TP4056, Basic_THT:TP4056, symbol Basic_SOP:TP4056
Connections:
- net Col0: now also U1.20
- net Col1: now also U1.19
- net Col2: now also U1.18
- net Col3: now also U1.17
- net Col4: now also U1.16 (SCK)
- net Col5: now also U1.15 (MISO)
- net Col6: now also U1.14 (MOSI)
- net GND: now also JP11.1, JP12.1, JP13.2, JP15.2, U1.0 (GND), U1.23 (GND), U1.3 (GND), U1.4 (GND)
- net LED: now also U1.1 (TX)
- net Row0: now also U1.7
- net Row1: now also U1.8
- net Row2: now also U1.9
- net Row3: now also U1.10
- net Row4: now also U1.11
- net SCL: now also U1.6 (SCL)
- net SDA: now also U1.5 (SDA)
- net VCC: now also JP10.1, JP9.1, U1.21 (VCC), U1.24 (RAW)
- net data: now also U1.2 (RX)
- net ~RESET: now also U1.22 (RESET)
- net at J1.1 (Pin_1), JP8.2: now also JP4.2; no longer JP1.2
- net at J1.2 (Pin_2), JP7.2: now also JP3.2; no longer JP2.2
- net at J1.3 (Pin_3), JP6.2: now also JP2.2; no longer JP3.2
- net at J1.4 (Pin_4), JP5.2: now also JP1.2; no longer JP4.2
- new net: JP11.2, JP9.2, U37.1 (+)
- new net: JP10.2, JP12.2, U37.2 (-)
- new net: JP13.1, JP14.1, U37.3 (OUT+)
- new net: J3.1 (Pin_1), U37.4 (B+)
- new net: J3.2 (Pin_2), U37.5 (B-)
- new net: JP15.1, JP16.1, U37.6 (OUT-)
- new net Bat+: JP14.2, JP16.2, U1.25 (Bat+)
- no-connect marks 7 -> 4
Other:
- moved on the sheet: J1
